File: leuchtibrille/gschau.kicad_sch (KiCad schematic)
At the start: 68 parts

Commit message: Upload of working version
Parts:
- renumbered C115 to C10, C117 to C12, C118 to C13, C119 to C14, C120 to C15, C121 to C16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
